Commit message: Changed triskarino description robot model

File: triskarino_robot/src/triskarino_description/urdf/base.xacro (robot description, xacro)
@@ -20,9 +20,11 @@
 			<color rgba="1 1 1 1"/>
 		</material>
+        <origin rpy="${rpy}"/>
 	</visual>
 	<collision>
 		<geometry>
-			<mesh scale="${scale}" filename="package://triskarino_description/meshes/base.stl"/>
+			<mesh scale="${scale}" filename="package://triskarino_description/meshes/base_v2.stl"/>
 		</geometry>
+         <origin rpy="${rpy}"/>
 	</collision>
 	</link>
@@ -30,5 +32,5 @@
 		<parent link="origin_link" />
 		<child link="base_link" />
-		<origin xyz="${xyz}"  rpy="${rpy}"/>
+		<origin xyz="${xyz}"  rpy="0 0 0"/>
 	</joint>
 </xacro:macro>

File: triskarino_robot/src/triskarino_description/urdf/rim.urdf.xacro (robot description, xacro)
@@ -4,20 +4,20 @@
 <xacro:macro
 	name="rim_macro"
-	params="name color xyz rpy">
+	params="name color xyz rpy scale_factor">
 		<link name="rim_${name}_link">
 			<inertial>
 				<origin xyz="0 0 -0.000343"/>
-				<mass value="0.00835758"/>
+				<mass value="${0.00835758 * scale_factor * scale_factor * scale_factor}"/>
 				<inertia
-					ixx="6.63684e-07"
+					ixx="${6.63684e-07 * scale_factor * scale_factor * scale_factor * scale_factor * scale_factor}"
 					ixy="0"
 					ixz="0"
-					iyy="6.63684e-07"
+					iyy="${6.63684e-07 * scale_factor * scale_factor * scale_factor * scale_factor * scale_factor}"
 					iyz="0"
-					izz="9.40333e-07"/>
+					izz="${9.40333e-07 * scale_factor * scale_factor * scale_factor * scale_factor * scale_factor}"/>
 			</inertial>
 			<visual>
 				<geometry>
-					<mesh filename="package://triskarino_description/meshes/rim.stl"/>
+					<mesh scale="${scale_factor} ${scale_factor} ${scale_factor}" filename="package://triskarino_description/meshes/rim.stl"/>
 				</geometry>
 				<material name="rim_${name}_material">
@@ -27,5 +27,5 @@
 			<collision>
 				<geometry>
-					<mesh filename="package://triskarino_description/meshes/rim.stl"/>
+					<mesh scale="${scale_factor} ${scale_factor} ${scale_factor}" filename="package://triskarino_description/meshes/rim.stl"/>
 				</geometry>
 			</collision>
@@ -44,4 +44,5 @@
 			xyz="0.01355 0 0.0055"
 			rpy="-1.570796326794896 0 0"
+            scale_factor="${scale_factor}"
 		/>
 		<xacro:roller_macro
@@ -50,4 +51,5 @@
 			xyz="0.00958129689 0.00958129689 -0.0055"
 			rpy="-1.570796326794896 0 0.7853981633974483"
+            scale_factor="${scale_factor}"
 		/>
 		<xacro:roller_macro
@@ -56,4 +58,5 @@
 			xyz="0 0.01355 0.0055"
 			rpy="-1.570796326794896 0 1.570796326794896"
+            scale_factor="${scale_factor}"
 		/>
 		<xacro:roller_macro
@@ -62,4 +65,5 @@
 			xyz="-0.00958129689 0.00958129689 -0.0055"
 			rpy="-1.570796326794896 0 2.356194490192345"
+            scale_factor="${scale_factor}"
 		/>
 		<xacro:roller_macro
@@ -68,4 +72,5 @@
 			xyz="-0.01355 0 0.0055"
 			rpy="-1.570796326794896 0 3.141592653589793"
+            scale_factor="${scale_factor}"
 		/>
 		<xacro:roller_macro
@@ -74,4 +79,5 @@
 			xyz="-0.00958129689 -0.00958129689 -0.0055"
 			rpy="-1.570796326794896 0 -2.356194490192345"
+            scale_factor="${scale_factor}"
 		/>
 		<xacro:roller_macro
@@ -80,4 +86,5 @@
 			xyz="0 -0.01355 0.0055"
 			rpy="-1.570796326794896 0 -1.570796326794896"
+            scale_factor="${scale_factor}"
 		/>
 		<xacro:roller_macro
@@ -86,4 +93,5 @@
 			xyz="0.00958129689 -0.00958129689 -0.0055"
 			rpy="-1.570796326794896 0 -0.7853981633974483"
+            scale_factor="${scale_factor}"
 		/>
 		<transmission name="rim_${name}_transmission">

File: triskarino_robot/src/triskarino_description/urdf/roller.urdf.xacro (robot description, xacro)
@@ -1,21 +1,22 @@
 <?xml version="1.0" ?>
 <robot xmlns:xacro="http://www.ros.org/wiki/xacro">
+<!-- SCALING OF MASS AND INERTIAL MATRICES ACCORDING TO https://answers.ros.org/question/237421/calculating-inertial-matrix-for-gazebo/ -->
 <xacro:macro
 	name="roller_macro"
-	params="parent name xyz rpy">
+	params="parent name xyz rpy scale_factor">
 		<link name="roller_${name}_rim_${parent}_link">
 			<inertial>
-				<mass value="0.00113845"/>
+				<mass value="${0.00113845 * scale_factor * scale_factor * scale_factor}"/>
 				<inertia
-					ixx="2.53776e-08"
+					ixx="${2.53776e-08 *scale_factor * scale_factor * scale_factor * scale_factor * scale_factor}"
 					ixy="0"
 					ixz="0"
-					iyy="2.53776e-08"
+					iyy="${2.53776e-08 *scale_factor * scale_factor * scale_factor * scale_factor * scale_factor}"
 					iyz="0"
-					izz="1.47666e-08"/>
+					izz="${1.47666e-08 * scale_factor * scale_factor * scale_factor * scale_factor * scale_factor}"/>
 			</inertial>
 			<visual>
 				<geometry>
-					<mesh filename="package://triskarino_description/meshes/roller.stl"/>
+					<mesh scale="${scale_factor} ${scale_factor} ${scale_factor}" filename="package://triskarino_description/meshes/roller.stl"/>
 				</geometry>
 				<material name="roller_material">
@@ -25,5 +26,5 @@
 			<collision>
 				<geometry>
-					<mesh filename="package://triskarino_description/meshes/roller.stl"/>
+					<mesh scale="${scale_factor} ${scale_factor} ${scale_factor}" filename="package://triskarino_description/meshes/roller.stl"/>
 				</geometry>
 			</collision>

File: triskarino_robot/src/triskarino_description/urdf/triskarino_core.xacro (robot description, xacro)
@@ -2,34 +2,59 @@
 <robot xmlns:xacro="http://www.ros.org/wiki/xacro" name="open_base">
 	<xacro:include filename="$(find triskarino_description)/urdf/rim.urdf.xacro"/>
-	<xacro:include filename="$(find triskarino_description)/urdf/triskarino_cover.xacro"/>
     <xacro:include filename="$(find triskarino_description)/urdf/base.xacro"/>
+    <xacro:include filename="$(find triskarino_description)/urdf/triskarino_top.xacro"/>
+    <xacro:include filename="$(find triskarino_description)/urdf/materials.xacro"/>
     <link name="origin_link"/>
+    <!-- BASE PLATE -->
     <xacro:base
         xyz="0 0 0.01905"
         scale="1 1 1"
-        rpy="0 1 0"
+        rpy="0 3.14 -0.05"
         />
+    <!-- LEFT WHEEL -->
 	<xacro:rim_macro
 		name="left"
 		color="0.3 0 0"
-		xyz="-0.03464101615 0.02 0"
-		rpy="1.570796326794896 0 1.047197551196597"/>
+		xyz="-0.1299038106 0.075 -0.02"
+		rpy="1.570796326794896 0 1.047197551196597"
+        scale_factor="2.0"/>
+    <!-- BACK WHEEL -->
 	<xacro:rim_macro
 		name="back"
 		color="0 0.3 0"
-		xyz="0 -0.04 0"
-		rpy="1.570796326794896 0 3.141592653589793"/>
+		xyz="0 -0.15 -0.02"
+		rpy="1.570796326794896 0 3.141592653589793"
+        scale_factor="2.0"/>
+    <!-- RIGHT WHEEL -->
 	<xacro:rim_macro
 		name="right"
 		color="0 0 0.3"
-		xyz="0.03464101615 0.02 0"
-		rpy="1.570796326794896 0 -1.047197551196597"/>
-    <xacro:cover
-        xyz="0 0 0"
-        rpy ="0 0 0"
-        scale="0.01 0.01 0.001"
-        color="base_material"
+		xyz="0.1299038106 0.075 -0.02"
+		rpy="1.570796326794896 0 -1.047197551196597"
+        scale_factor="2.0"/>
+    <!-- FIRST CYLINDER SET AT THE BASE OF THE LIDAR -->
+    <xacro:top
+        name="layer_0"
+        xyz="0 0 0.03"
+        rpy="0 0 0"
         parent="base_link"
-    />
+        color="grey"
+        radius="0.2"
+        length="0.01"
+        mass="0.001"
+        />
+    <!-- LIDAR -->
+    <xacro:include filename="lidar.xacro" />
+    <!-- SECOND CYLINDER MAKING UP THE TOP OF THE ROBOT -->
+    <xacro:top
+        name="layer_1"
+        xyz="0 0 0.31"
+        rpy="0 0 0"
+        parent="base_link"
+        color="blue"
+        radius="0.2"
+        length="0.4"
+        mass="0.01"
+        />
 	<gazebo reference="base_link">
     		<material>Gazebo/White</material>

File: triskarino_robot/src/triskarino_description/urdf/triskarino_top.xacro (robot description, xacro)
@@ -1,11 +1,12 @@
 <?xml version="1.0"?>
 <robot xmlns:xacro="http://www.ros.org/wiki/xacro" >
-<xacro:macro name="top" params="xyz rpy parent color radius length mass">
-    <joint name="top_joint" type="fixed">
+<xacro:include filename="$(find triskarino_description)/urdf/inertial_macros.xacro"/>
+<xacro:macro name="top" params="xyz name rpy parent color radius length mass">
+    <joint name="${name}_joint" type="fixed">
         <parent link="${parent}"/>
-        <child link="top_link"/>
+        <child link="${name}_link"/>
         <origin xyz="${xyz}" rpy="${rpy}" />
     </joint>
-    <link name="top_link">
+    <link name="${name}_link">
         <visual>
             <geometry>
