Commit message: Triskarino description rviz now working with lidar and omni_teleop, integrated hokuyo lidar

File: triskarino_robot/triskarino_description/urdf/materials.xacro (robot description, xacro)
@@ -16,4 +16,7 @@
     <color rgba="${255/255} ${108/255} ${10/255} 1.0"/>
   </material>
+  <material name="dark_grey">
+    <color rgba="${220/255} ${220/255} ${220/255} 1.0"/>
+  </material>
   <material name="brown">
     <color rgba="${222/255} ${207/255} ${195/255} 1.0"/>

File: triskarino_robot/triskarino_description/urdf/rim.urdf.xacro (robot description, xacro)
@@ -5,4 +5,10 @@
 	name="rim_macro"
 	params="name color xyz rpy scale_factor">
+		<joint name="rim_${name}_joint" type="continuous">
+			<parent link="base_link" />
+			<child link="rim_${name}_link"/>
+			<axis xyz="0 0 1"/>
+			<origin xyz="${xyz}" rpy="${rpy}"/>
+		</joint>
 		<link name="rim_${name}_link">
 			<inertial>
@@ -31,14 +37,6 @@
 			</collision>
 		</link>
-		<joint
-			name="rim_${name}_joint"
-			type="continuous">
-			<parent link="base_link" />
-			<child link="rim_${name}_link" />
-			<axis xyz="0 0 1"/>
-			<origin xyz="${xyz}" rpy="${rpy}"/>
-		</joint>
 		<xacro:roller_macro
-			parent="${name}"
+			parent="rim_${name}_link"
 			name="e"
 			xyz="0.01355 0 0.0055"
@@ -47,5 +45,5 @@
 		/>
 		<xacro:roller_macro
-			parent="${name}"
+			parent="rim_${name}_link"
 			name="ne"
 			xyz="0.00958129689 0.00958129689 -0.0055"
@@ -54,5 +52,5 @@
 		/>
 		<xacro:roller_macro
-			parent="${name}"
+			parent="rim_${name}_link"
 			name="n"
 			xyz="0 0.01355 0.0055"
@@ -61,5 +59,5 @@
 		/>
 		<xacro:roller_macro
-			parent="${name}"
+			parent="rim_${name}_link"
 			name="nw"
 			xyz="-0.00958129689 0.00958129689 -0.0055"
@@ -68,5 +66,5 @@
 		/>
 		<xacro:roller_macro
-			parent="${name}"
+			parent="rim_${name}_link"
 			name="w"
 			xyz="-0.01355 0 0.0055"
@@ -75,5 +73,5 @@
 		/>
 		<xacro:roller_macro
-			parent="${name}"
+			parent="rim_${name}_link"
 			name="sw"
 			xyz="-0.00958129689 -0.00958129689 -0.0055"
@@ -82,5 +80,5 @@
 		/>
 		<xacro:roller_macro
-			parent="${name}"
+			parent="rim_${name}_link"
 			name="s"
 			xyz="0 -0.01355 0.0055"
@@ -89,5 +87,5 @@
 		/>
 		<xacro:roller_macro
-			parent="${name}"
+			parent="rim_${name}_link"
 			name="se"
 			xyz="0.00958129689 -0.00958129689 -0.0055"

File: triskarino_robot/triskarino_description/urdf/roller.urdf.xacro (robot description, xacro)
@@ -5,5 +5,5 @@
 	name="roller_macro"
 	params="parent name xyz rpy scale_factor">
-		<link name="roller_${name}_rim_${parent}_link">
+		<link name="roller_${name}_${parent}_link">
 			<inertial>
 				<mass value="${0.00113845 * scale_factor * scale_factor * scale_factor}"/>
@@ -30,10 +30,10 @@
 			</collision>
 		</link>
-	<gazebo reference="roller_${name}_rim_${parent}_link">
+	<gazebo reference="roller_${name}_{parent}">
     		<material>Gazebo/Black</material>
   	</gazebo>
-		<joint name="roller_${name}_rim_${parent}_joint" type="continuous">
-			<parent link="rim_${parent}_link"/>
-			<child link="roller_${name}_rim_${parent}_link"/>
+		<joint name="roller_${name}_${parent}_joint" type="continuous">
+			<parent link="${parent}"/>
+			<child link="roller_${name}_${parent}_link"/>
 			<axis xyz="0 0 1"/>
 			<origin xyz="${xyz}" rpy="${rpy}"/>

File: triskarino_robot/triskarino_description/urdf/triskarino.urdf.xacro (robot description, xacro)
@@ -1,4 +1,4 @@
 <?xml version="1.0"?>
-<robot xmlns:xacro="http://www.ros.org/wiki/xacro"  name="robot">
+<robot xmlns:xacro="http://www.ros.org/wiki/xacro"  name="triskarino">
     <xacro:include filename="triskarino_core.xacro" />
 </robot>

File: triskarino_robot/triskarino_description/urdf/triskarino_core.xacro (robot description, xacro)
@@ -1,8 +1,9 @@
 <?xml version="1.0"?>
-<robot xmlns:xacro="http://www.ros.org/wiki/xacro" name="open_base">
+<robot xmlns:xacro="http://www.ros.org/wiki/xacro" name="triskarino">
 	<xacro:include filename="$(find triskarino_description)/urdf/rim.urdf.xacro"/>
     <xacro:include filename="$(find triskarino_description)/urdf/base.xacro"/>
     <xacro:include filename="$(find triskarino_description)/urdf/triskarino_top.xacro"/>
     <xacro:include filename="$(find triskarino_description)/urdf/materials.xacro"/>
+    <xacro:include filename="$(find triskarino_description)/urdf/hokuyo.xacro"/>
     <link name="origin_link"/>
     <!-- BASE PLATE -->
@@ -44,6 +45,10 @@
         mass="0.001"
         />
-    <!-- LIDAR -->
-    <xacro:include filename="lidar.xacro" />
+    <xacro:hokuyo_ust10_mount
+        topic="scan"
+        parent_link="layer_0_link"
+        xyz="0 0.11 0"
+        rpy="0 0 1.5708"
+    />
     <!-- SECOND CYLINDER MAKING UP THE TOP OF THE ROBOT -->
     <xacro:top
@@ -71,5 +76,5 @@
 	<gazebo>
 		<plugin name="gazebo_ros_control" filename="libgazebo_ros_control.so">
-		<robotNamespace>/open_base</robotNamespace>
+		<robotNamespace>/triskarino</robotNamespace>
 		</plugin>
 	</gazebo>
