Commit message: Adding changes triskarino_navigation, description and hw

File: triskarino_robot/triskarino_description/urdf/hokuyo.xacro (robot description, xacro)
@@ -2,7 +2,7 @@
 <robot xmlns:xacro="http://ros.org/wiki/xacro">
   <xacro:macro name="hokuyo_ust10_mount" params="topic parent_link min_angle:=-2.0944 max_angle:=2.0944 xyz rpy">
-    <xacro:macro name="hokuyo_ust10" params="frame:=laser topic:=scan sample_size:=720 update_rate:=50
-               min_angle:=${min_angle} max_angle:=${max_angle} min_range:=0.01 max_range:=30 robot_namespace:=triskarino/">
-      <link name="${frame}">
+    <xacro:macro name="hokuyo_ust10" params="frame:=laser topic:=scan sample_size:=720 update_rate:=10.0
+               min_angle:=${min_angle} max_angle:=${max_angle} min_range:=0.01 max_range:=30 robot_namespace:=triskarino ">
+      <link name="laser">
         <inertial>
           <mass value="1.1" />
@@ -13,5 +13,5 @@
         </inertial>
       </link>
-      <gazebo reference="${frame}">
+      <gazebo reference="laser">
         <turnGravityOff>true</turnGravityOff>
         <sensor type="ray" name="${frame}">
@@ -39,10 +39,9 @@
             </noise>
           </ray>
-          <plugin name="laser_controller" filename="libgazebo_ros_ray_sensor.so">
-            <ros>
-                <argument>~/out:=scan</argument>
-            </ros>
-            <output_type>sensor_msgs/LaserScan</output_type>
-            <frame_name>laser</frame_name>
+          <plugin name="laser_controller" filename="libgazebo_ros_laser.so">
+            <tf_prefix></tf_prefix>
+            <frameName>${frame}</frameName>
+            <topicName>${topic}</topicName>
+            <robotNamespace>triskarino</robotNamespace>
           </plugin>
         </sensor>
@@ -60,5 +59,5 @@
         <geometry>
           <!-- Origin of this mesh is the base of the bracket. -->
-          <mesh filename="package://urg_node/meshes/hokuyo_ust10.stl" />
+          <mesh filename="package://triskarino_description/meshes/hokuyo_ust10.stl" />
         </geometry>
         <material name="dark_grey" />
@@ -71,4 +70,5 @@
       <child link="laser" />
     </joint>
+    <!-- Fix to make rviz laserscan work! -->
     <gazebo reference="laser_mount">
       <material>Gazebo/DarkGrey</material>

File: triskarino_robot/triskarino_description/urdf/rim.urdf.xacro (robot description, xacro)
@@ -2,9 +2,10 @@
 <robot xmlns:xacro="http://www.ros.org/wiki/xacro">
 <xacro:include filename="$(find triskarino_description)/urdf/roller.urdf.xacro"/>
+<xacro:include filename="$(find triskarino_description)/urdf/inertial_macros.xacro"/>
 <xacro:macro
 	name="rim_macro"
-	params="name color xyz rpy scale_factor">
+	params="name color xyz rpy">
 		<joint name="rim_${name}_joint" type="continuous">
-			<parent link="base_link" />
+			<parent link="plate_link" />
 			<child link="rim_${name}_link"/>
 			<axis xyz="0 0 1"/>
@@ -13,17 +14,11 @@
 		<link name="rim_${name}_link">
 			<inertial>
-				<origin xyz="0 0 -0.000343"/>
-				<mass value="${0.00835758 * scale_factor * scale_factor * scale_factor}"/>
-				<inertia
-					ixx="${6.63684e-07 * scale_factor * scale_factor * scale_factor * scale_factor * scale_factor}"
-					ixy="0"
-					ixz="0"
-					iyy="${6.63684e-07 * scale_factor * scale_factor * scale_factor * scale_factor * scale_factor}"
-					iyz="0"
-					izz="${9.40333e-07 * scale_factor * scale_factor * scale_factor * scale_factor * scale_factor}"/>
-			</inertial>
+				<origin xyz="-0.00000435 -0.00000262 -0.00011790"/>
+				<mass value="0.20000000"/>
+				<inertia ixx="0.00005620" ixy="-0.00000000" ixz="0.00000000" iyy="0.00005620" iyz="-0.00000000" izz="0.00007735"/>
+			  </inertial>
 			<visual>
 				<geometry>
-					<mesh scale="${scale_factor} ${scale_factor} ${scale_factor}" filename="package://triskarino_description/meshes/rim.stl"/>
+					<mesh filename="package://triskarino_description/meshes/rim_scaled.stl"/>
 				</geometry>
 				<material name="rim_${name}_material">
@@ -32,7 +27,11 @@
 			</visual>
 			<collision>
+				<origin xyz="0 0 0" rpy="0 0 0" />
 				<geometry>
-					<mesh scale="${scale_factor} ${scale_factor} ${scale_factor}" filename="package://triskarino_description/meshes/rim.stl"/>
+					<cylinder length="0.02" radius="0.032" />
 				</geometry>
+				<surface>
+					<bounce restitution_coefficient="0.0001" />
+				</surface>
 			</collision>
 		</link>
@@ -42,5 +41,4 @@
 			xyz="0.01355 0 0.0055"
 			rpy="-1.570796326794896 0 0"
-            scale_factor="${scale_factor}"
 		/>
 		<xacro:roller_macro
@@ -49,5 +47,4 @@
 			xyz="0.00958129689 0.00958129689 -0.0055"
 			rpy="-1.570796326794896 0 0.7853981633974483"
-            scale_factor="${scale_factor}"
 		/>
 		<xacro:roller_macro
@@ -56,5 +53,4 @@
 			xyz="0 0.01355 0.0055"
 			rpy="-1.570796326794896 0 1.570796326794896"
-            scale_factor="${scale_factor}"
 		/>
 		<xacro:roller_macro
@@ -63,5 +59,4 @@
 			xyz="-0.00958129689 0.00958129689 -0.0055"
 			rpy="-1.570796326794896 0 2.356194490192345"
-            scale_factor="${scale_factor}"
 		/>
 		<xacro:roller_macro
@@ -70,5 +65,4 @@
 			xyz="-0.01355 0 0.0055"
 			rpy="-1.570796326794896 0 3.141592653589793"
-            scale_factor="${scale_factor}"
 		/>
 		<xacro:roller_macro
@@ -77,5 +71,4 @@
 			xyz="-0.00958129689 -0.00958129689 -0.0055"
 			rpy="-1.570796326794896 0 -2.356194490192345"
-            scale_factor="${scale_factor}"
 		/>
 		<xacro:roller_macro
@@ -84,5 +77,4 @@
 			xyz="0 -0.01355 0.0055"
 			rpy="-1.570796326794896 0 -1.570796326794896"
-            scale_factor="${scale_factor}"
 		/>
 		<xacro:roller_macro
@@ -91,5 +83,4 @@
 			xyz="0.00958129689 -0.00958129689 -0.0055"
 			rpy="-1.570796326794896 0 -0.7853981633974483"
-            scale_factor="${scale_factor}"
 		/>
 		<transmission name="rim_${name}_transmission">
@@ -103,4 +94,27 @@
 			</actuator>
 		</transmission>
+	<gazebo reference="rim_${name}_link">
+		<collision name="rim_${name}_link_collision">
+			<surface>
+			  <contact>
+                <ode>
+                  <kp>1e+6</kp>
+                  <kd>1</kd>
+                  <min_depth>0.00001</min_depth>
+                </ode>
+			  </contact>
+			  <friction>
+				<ode>
+				<mu>0</mu>
+				<mu2>0</mu2>
+				<max_contacts>2</max_contacts>
+				<fdir1>0 0 1</fdir1>
+				<slip1>1</slip1>
+				<slip2>1</slip2>
+				</ode>
+			  </friction>
+			</surface>
+		  </collision>
+  	</gazebo>
 	</xacro:macro>
 </robot>

File: triskarino_robot/triskarino_description/urdf/roller.urdf.xacro (robot description, xacro)
@@ -4,19 +4,14 @@
 <xacro:macro
 	name="roller_macro"
-	params="parent name xyz rpy scale_factor">
+	params="parent name xyz rpy">
 		<link name="roller_${name}_${parent}_link">
 			<inertial>
-				<mass value="${0.00113845 * scale_factor * scale_factor * scale_factor}"/>
-				<inertia
-					ixx="${2.53776e-08 *scale_factor * scale_factor * scale_factor * scale_factor * scale_factor}"
-					ixy="0"
-					ixz="0"
-					iyy="${2.53776e-08 *scale_factor * scale_factor * scale_factor * scale_factor * scale_factor}"
-					iyz="0"
-					izz="${1.47666e-08 * scale_factor * scale_factor * scale_factor * scale_factor * scale_factor}"/>
-			</inertial>
+				<origin xyz="0.00000004 -0.00000000 -0.00000002"/>
+				<mass value="0.05000000"/>
+				<inertia ixx="0.00000328" ixy="0.00000000" ixz="-0.00000000" iyy="0.00000328" iyz="-0.00000000" izz="0.00000191"/>
+			  </inertial>
 			<visual>
 				<geometry>
-					<mesh scale="${scale_factor} ${scale_factor} ${scale_factor}" filename="package://triskarino_description/meshes/roller.stl"/>
+					<mesh filename="package://triskarino_description/meshes/roller_scaled.stl"/>
 				</geometry>
 				<material name="roller_material">
@@ -26,5 +21,5 @@
 			<collision>
 				<geometry>
-					<mesh scale="${scale_factor} ${scale_factor} ${scale_factor}" filename="package://triskarino_description/meshes/roller.stl"/>
+					<mesh filename="package://triskarino_description/meshes/roller_scaled.stl"/>
 				</geometry>
 			</collision>
@@ -39,4 +34,12 @@
 			<origin xyz="${xyz}" rpy="${rpy}"/>
 		</joint>
+		<gazebo reference="roller_${name}_${parent}_link">
+			<mu1 value="0.0"/>
+			<mu2 value="0.0"/>
+			<minDepth>0.001</minDepth>
+			<kp value="1000000"/>
+			<kd value="1"/>
+			<maxContacts value= "0"/>
+		</gazebo>
 	</xacro:macro>
 </robot>

File: triskarino_robot/triskarino_description/urdf/triskarino_core.xacro (robot description, xacro)
@@ -2,46 +2,63 @@
 <robot xmlns:xacro="http://www.ros.org/wiki/xacro" name="triskarino">
 	<xacro:include filename="$(find triskarino_description)/urdf/rim.urdf.xacro"/>
-    <xacro:include filename="$(find triskarino_description)/urdf/base.xacro"/>
-    <xacro:include filename="$(find triskarino_description)/urdf/triskarino_top.xacro"/>
+    <xacro:include filename="$(find triskarino_description)/urdf/base.urdf.xacro"/>
+    <xacro:include filename="$(find triskarino_description)/urdf/triskarino_cylinder.xacro"/>
     <xacro:include filename="$(find triskarino_description)/urdf/materials.xacro"/>
     <xacro:include filename="$(find triskarino_description)/urdf/hokuyo.xacro"/>
-    <link name="origin_link"/>
+    <link name="base_link"/>
     <!-- BASE PLATE -->
     <xacro:base
-        xyz="0 0 0.01905"
-        scale="1 1 1"
-        rpy="0 3.14 -0.05"
+        xyz="0 0 0.1"
+        scale_factor="0.001"
+        rpy="0 3.14 0"
         />
+    <joint name="base_footprint_joint" type="fixed">
+        <parent link="base_link"/>
+        <child link="base_footprint"/>
+        <origin xyz="0 0 0" rpy="0 0 0"/>
+    </joint>
+    <link name="base_footprint"></link>
     <!-- LEFT WHEEL -->
 	<xacro:rim_macro
 		name="left"
 		color="0.3 0 0"
-		xyz="-0.1299038106 0.075 -0.02"
+		xyz="-0.142894191624 0.0825 -0.035"
 		rpy="1.570796326794896 0 1.047197551196597"
-        scale_factor="2.0"/>
+        />
     <!-- BACK WHEEL -->
 	<xacro:rim_macro
 		name="back"
 		color="0 0.3 0"
-		xyz="0 -0.15 -0.02"
+		xyz="0 -0.1650 -0.035"
 		rpy="1.570796326794896 0 3.141592653589793"
-        scale_factor="2.0"/>
+        />
     <!-- RIGHT WHEEL -->
 	<xacro:rim_macro
 		name="right"
 		color="0 0 0.3"
-		xyz="0.1299038106 0.075 -0.02"
+		xyz="0.142894191624 0.0825 -0.035"
 		rpy="1.570796326794896 0 -1.047197551196597"
-        scale_factor="2.0"/>
+        />
+    <!-- CYLINDER USED AS AXIS FOR THE ROBOT, Z HAS TO BE ADJUSTED ACCORDING TO THE LENGTH OF THE AXIS -->
+    <xacro:cylinder
+        name="axis"
+        xyz="0 0 0.2"
+        rpy="0 0 0"
+        parent="plate_link"
+        color="grey"
+        radius="0.01"
+        length="0.4"
+        mass="1"
+        />
     <!-- FIRST CYLINDER SET AT THE BASE OF THE LIDAR -->
-    <xacro:top
+    <xacro:cylinder
         name="layer_0"
-        xyz="0 0 0.03"
+        xyz="0 0 -0.17"
         rpy="0 0 0"
-        parent="base_link"
+        parent="axis_link"
         color="grey"
         radius="0.2"
         length="0.01"
-        mass="0.001"
+        mass="1"
         />
     <xacro:hokuyo_ust10_mount
@@ -51,31 +68,19 @@
         rpy="0 0 1.5708"
     />
-    <!-- SECOND CYLINDER MAKING UP THE TOP OF THE ROBOT -->
-    <xacro:top
-        name="layer_1"
-        xyz="0 0 0.31"
-        rpy="0 0 0"
-        parent="base_link"
-        color="blue"
-        radius="0.2"
-        length="0.4"
-        mass="0.01"
-        />
-	<gazebo reference="base_link">
+	<gazebo reference="plate_link">
     		<material>Gazebo/White</material>
   	</gazebo>
-	<gazebo reference="rim_left_link">
-    		<material>Gazebo/Red</material>
-  	</gazebo>
-	<gazebo reference="rim_back_link">
-    		<material>Gazebo/Green</material>
-  	</gazebo>
-	<gazebo reference="rim_right_link">
-    		<material>Gazebo/Blue</material>
+    <gazebo reference="base_link">
+		<mu1 value="0.0"/>
+		<mu2 value="0.0"/>
   	</gazebo>
 	<gazebo>
-		<plugin name="gazebo_ros_control" filename="libgazebo_ros_control.so">
-		<robotNamespace>/triskarino</robotNamespace>
-		</plugin>
-	</gazebo>
+        <plugin name="triskarino_controller" filename="libgazebo_ros_planar_move.so">
+            <commandTopic>/cmd_vel</commandTopic>
+            <odometryTopic>/odom</odometryTopic>
+            <odometryFrame>/odom</odometryFrame>
+            <odometryRate>50.0</odometryRate>
+            <robotBaseFrame>base_link</robotBaseFrame>
+        </plugin>
+    </gazebo>
 </robot>
